File: boards/aac/aac.kicad_sch (KiCad schematic)
At the start: 76 parts, among them J1 Conn_01x15, J2 Conn_01x15, Q1 CMPT930, Q2 CMPT930, Q3 CMPT930, Q4 CMPT930, Q5 CMPT930, Q6 CMPT930, Q7 BC847C, T1 1:2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

Commit message: Add PSA switching modules and rework fine ref
Parts:
- C12: value 0.0033uF -> 0.033uF
- R2: value NOM -> 4700
- R32, R36: value 3320 -> 3300
Changed lines of the file:
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@@
 			)
 		)
-		(property "Value" "3320"
+		(property "Value" "3300"
 			(at 240.03 158.75 90)
 			(effects
@@
 			)
 		)
-		(property "Value" "3320"
+		(property "Value" "3300"
 			(at 247.65 213.36 0)
 			(effects
@@
 			)
 		)
-		(property "Value" "0.0033uF"
+		(property "Value" "0.033uF"
 			(at 262.382 218.44 90)
 			(effects
@@
 			)
 		)
-		(property "Value" "NOM"
+		(property "Value" "4700"
 			(at 133.35 127 0)
 			(effects
