File: boards/agc/p.kicad_sch (KiCad schematic)
At the start: 2 parts

Commit message: Add PSA switching modules and rework fine ref
Changed lines of the file:
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@@
 (kicad_sch
-	(version 20231120)
+	(version 20250114)
 	(generator "eeschema")
-	(generator_version "8.0")
+	(generator_version "9.0")
 	(paper "A4")
 	(junction
@@
 		(shape output)
 		(at 138.43 81.28 0)
-		(fields_autoplaced yes)
 		(effects
 			(font
@@
 		(shape input)
 		(at 119.38 81.28 180)
-		(fields_autoplaced yes)
 		(effects
 			(font
