File: boards/fine_ref/fine_ref.kicad_sch (KiCad schematic)
At the start: 7 parts, among them J1 Conn_01x15, J2 Conn_01x15, T1 109R

Commit message: Add PSA switching modules and rework fine ref
Parts:
- added TP1, TP2, TP3, TP4: TestPoint, TestPoint:TestPoint_Keystone_5000-5004_Miniature, symbol Connector:TestPoint
Connections:
- net 28_HI: now also TP1.1
- net 28_LO: now also TP2.1
- net 5_HI: now also J2.5 (Pin_5), J2.6 (Pin_6), J2.7 (Pin_7), TP3.1; no longer J2.10 (Pin_10), J2.11 (Pin_11), J2.9 (Pin_9)
- net 5_LO: now also J2.10 (Pin_10), J2.9 (Pin_9), TP4.1; no longer J2.6 (Pin_6), J2.7 (Pin_7)
