File: boards/aux_relays/aux_relays.kicad_sch (KiCad schematic)
At the start: 44 parts, among them J1 Conn_01x15, J2 Conn_01x15, K1 EC2-24NU, K2 EC2-24NU, K3 EC2-24NU, K4 EC2-24NU, K5 EC2-24NU, Q1 MMBT2907, SW1 SW_SPDT, SW2 SW_SPDT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

Commit message: Corrected switch layouts for auxiliary relays and LM switching boards
Parts:
- R6: value 1000 -> 4300
- R7: value 1000 -> 100
Connections:
- net +28V: now also SW1.3 (C); no longer SW1.1 (A)
- net CAGE: now also CR1.2 (A), CR5.2 (A), J1.7 (Pin_7), SW1.2 (B); no longer J2.2 (Pin_2), K5.5
- net GND: no longer J1.7 (Pin_7)
- net at SW3.1 (A): no longer R8.1
- net at SW3.3 (C): now also R8.1
- net at R6.1, R7.1: now also SW2.3 (C); no longer SW2.1 (A)
- new net CDU_CAGE: J2.2 (Pin_2), K5.5
Other:
- moved on the sheet: R6, R7, R8, SW1
