File: boards/lm_switching/lm_switching.kicad_sch (KiCad schematic)
At the start: 13 parts, among them J1 Conn_01x15, J2 Conn_01x15, SW1 SW_3PDT

Commit message: Corrected switch layouts for auxiliary relays and LM switching boards
Connections:
- net ATCA_800CPS_HI: now also SW1.4 (A); no longer SW1.6 (C)
- net ATCA_800CPS_LO: now also SW1.7 (A); no longer SW1.9 (C)
- net PGNCS_800CPS_HI: now also SW1.6 (C); no longer SW1.4 (A)
- net PGNCS_800CPS_LO: now also SW1.9 (C); no longer SW1.7 (A)
- net RD874: now also SW1.3 (C); no longer SW1.1 (A)
Changed lines of the file:
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@@
 	)
 	(no_connect
-		(at 111.76 58.42)
+		(at 111.76 53.34)
 	)
 	(no_connect
@@
 	(wire
 		(pts
-			(xy 92.71 53.34) (xy 111.76 53.34)
+			(xy 92.71 58.42) (xy 111.76 58.42)
 		)
 		(stroke
@@
 	)
 	(label "PGNCS_800CPS_LO"
-		(at 92.71 73.66 0)
+		(at 92.71 78.74 0)
 		(effects
 			(font
@@
 	)
 	(label "RD874"
-		(at 92.71 53.34 0)
+		(at 92.71 58.42 0)
 		(effects
 			(font
@@
 	)
 	(label "ATCA_800CPS_HI"
-		(at 92.71 68.58 0)
+		(at 92.71 63.5 0)
 		(effects
 			(font
@@
 	)
 	(label "PGNCS_800CPS_HI"
-		(at 92.71 63.5 0)
+		(at 92.71 68.58 0)
 		(effects
 			(font
@@
 	)
 	(label "ATCA_800CPS_LO"
-		(at 92.71 78.74 0)
-		(effects
-			(font
+		(at 92.71 73.66 0)
+		(effects
+			(font
